File: DRV8701_2Motors.kicad_pcb (KiCad board)
At the start: 4 copper layers, 92 x 61 mm, 94 parts, among them J1 Conn_01x02, J10 Conn_01x04, J11 Conn_01x03, J2 Conn_01x10, J3 Conn_01x10, J4 Conn_01x02, J5 Conn_01x02, J6 Conn_01x04, J7 Conn_ST_STDC14, J8 Conn_01x03, J9 Conn_01x04, SW1 SW_SPDT_321, U16 STM32F303RETx, U3 AM26LV32xD, U4 AM26LV32xD

Commit message: final push
Parts:
- C16, C22: value 47u -> 10u; footprint Capacitor:Wurth-47u-63V -> Capacitor_SMD:C_0805_2012Metric
- moved C8 42.7 mm to (118.4, 118.1), turned to -135 degrees
- moved C16 17.8 mm to (166.2, 113.6), turned to 0 degrees
- moved U6 12.6 mm to (170.0, 107.8)
- moved U13 11.5 mm to (120.2, 105.5), turned to 90 degrees
- moved U8 10.4 mm to (170.0, 102.0), turned to -90 degrees
- moved C15 9.11 mm to (165.8, 111.9)
- moved U9 8.49 mm to (176.7, 105.3), turned to 0 degrees
- moved U11 8.41 mm to (120.2, 111.2)
- moved C22 8.08 mm to (123.9, 110.6), turned to 180 degrees
- moved U14 7.89 mm to (109.0, 105.6), turned to 0 degrees
- moved U12 6.84 mm to (112.8, 107.0), turned to 180 degrees
- moved C14 6.68 mm to (166.3, 110.4), turned to 90 degrees
- moved C13 5.36 mm to (166.1, 108.2), turned to 90 degrees
- moved C18 5.33 mm to (129.4, 105.6), turned to 0 degrees
- moved J5 5.00 mm to (102.8, 103.8), turned to -90 degrees
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- renumbered U13 to U12, U12 to U13, U8 to U7, U7 to U8
Connections:
- net Net-(U10-GH2) renamed /MoteurGauche/GH2
- net Net-(U5-GH2) renamed /MoteurDroit/GH2
- C16 pad 1: VDC -> GND
- C16 pad 2: GND -> VDC
- C22 pad 1: VDC -> GND
- C22 pad 2: GND -> VDC
- J4 pad 1: /MoteurDroit/SH2 -> /MoteurDroit/SH1
- J4 pad 2: /MoteurDroit/SH1 -> /MoteurDroit/SH2
- J5 pad 1: /MoteurGauche/SH2 -> /MoteurGauche/SH1
- J5 pad 2: /MoteurGauche/SH1 -> /MoteurGauche/SH2
- U10 pad 17: Net-(U10-GH1) -> /MoteurGauche/GH1
- U10 pad 19: Net-(U10-GL1) -> /MoteurGauche/GL1
- U10 pad 22: /MoteurGauche/SH2 -> /MoteurGauche/GL2
- U12 pad 1: /MoteurGauche/jonctionSS -> GND
- U12 pad 2: /MoteurGauche/jonctionSS -> GND
- U12 pad 3: /MoteurGauche/jonctionSS -> GND
- U12 pad 4: Net-(U10-GL1) -> /MoteurGauche/GL2
- U12 pad 5: /MoteurGauche/SH1 -> /MoteurGauche/SH2
- U12 pad 6: /MoteurGauche/SH1 -> /MoteurGauche/SH2
- U12 pad 7: /MoteurGauche/SH1 -> /MoteurGauche/SH2
- U12 pad 8: /MoteurGauche/SH1 -> /MoteurGauche/SH2
- U12 pad 9: /MoteurGauche/SH1 -> /MoteurGauche/SH2
- U13 pad 1: /MoteurGauche/jonctionSS -> /MoteurGauche/SH1
- U13 pad 2: /MoteurGauche/jonctionSS -> /MoteurGauche/SH1
- U13 pad 3: /MoteurGauche/jonctionSS -> /MoteurGauche/SH1
- U13 pad 4: /MoteurGauche/SH2 -> /MoteurGauche/GH1
- U13 pad 5: /MoteurGauche/SH2 -> VDC
- U13 pad 6: /MoteurGauche/SH2 -> VDC
- U13 pad 7: /MoteurGauche/SH2 -> VDC
- U13 pad 8: /MoteurGauche/SH2 -> VDC
- U13 pad 9: /MoteurGauche/SH2 -> VDC
- U14 pad 1: /MoteurGauche/SH1 -> GND
- U14 pad 2: /MoteurGauche/SH1 -> GND
- U14 pad 3: /MoteurGauche/SH1 -> GND
- U14 pad 4: Net-(U10-GH1) -> /MoteurGauche/GL1
- U14 pad 5: VDC -> /MoteurGauche/SH1
- U14 pad 6: VDC -> /MoteurGauche/SH1
- U14 pad 7: VDC -> /MoteurGauche/SH1
- U14 pad 8: VDC -> /MoteurGauche/SH1
- U14 pad 9: VDC -> /MoteurGauche/SH1
- U5 pad 17: Net-(U5-GH1) -> /MoteurDroit/GH1
- U5 pad 19: Net-(U5-GL1) -> /MoteurDroit/GL1
- U5 pad 22: /MoteurDroit/SH2 -> /MoteurDroit/GL2
- U7 pad 1: /MoteurDroit/jonctionSS -> GND
- U7 pad 2: /MoteurDroit/jonctionSS -> GND
- U7 pad 3: /MoteurDroit/jonctionSS -> GND
- U7 pad 4: Net-(U5-GL1) -> /MoteurDroit/GL2
- U7 pad 5: /MoteurDroit/SH1 -> /MoteurDroit/SH2
- U7 pad 6: /MoteurDroit/SH1 -> /MoteurDroit/SH2
- U7 pad 7: /MoteurDroit/SH1 -> /MoteurDroit/SH2
- U7 pad 8: /MoteurDroit/SH1 -> /MoteurDroit/SH2
- U7 pad 9: /MoteurDroit/SH1 -> /MoteurDroit/SH2
- U8 pad 1: /MoteurDroit/jonctionSS -> /MoteurDroit/SH1
- U8 pad 2: /MoteurDroit/jonctionSS -> /MoteurDroit/SH1
- U8 pad 3: /MoteurDroit/jonctionSS -> /MoteurDroit/SH1
- U8 pad 4: /MoteurDroit/SH2 -> /MoteurDroit/GH1
- U8 pad 5: /MoteurDroit/SH2 -> VDC
- U8 pad 6: /MoteurDroit/SH2 -> VDC
- U8 pad 7: /MoteurDroit/SH2 -> VDC
- U8 pad 8: /MoteurDroit/SH2 -> VDC
- U8 pad 9: /MoteurDroit/SH2 -> VDC
- U9 pad 1: /MoteurDroit/SH1 -> GND
- U9 pad 2: /MoteurDroit/SH1 -> GND
- U9 pad 3: /MoteurDroit/SH1 -> GND
- U9 pad 4: Net-(U5-GH1) -> /MoteurDroit/GL1
- U9 pad 5: VDC -> /MoteurDroit/SH1
- U9 pad 6: VDC -> /MoteurDroit/SH1
- U9 pad 7: VDC -> /MoteurDroit/SH1
- U9 pad 8: VDC -> /MoteurDroit/SH1
- U9 pad 9: VDC -> /MoteurDroit/SH1
Routing:
- net /MoteurDroit/GL2: track 0.00 -> 22.8 mm, vias 0 -> 2
- net /MoteurDroit/GH1: track 0.00 -> 22.5 mm, vias 0 -> 2
- net /MoteurDroit/GL1: track 0.00 -> 20.8 mm, vias 0 -> 2
- net Net-(U10-GH1): track 18.3 -> 0.00 mm
- net Net-(U5-GH1): track 18.1 -> 0.00 mm
- net /MoteurGauche/GL1: track 0.00 -> 17.7 mm
- net /MoteurGauche/GL2: track 0.00 -> 14.7 mm, vias 0 -> 2
- net /MoteurGauche/GH1: track 0.00 -> 13.2 mm, vias 0 -> 2
- net /MoteurGauche/SH2: track 23.6 -> 10.6 mm, vias 11 -> 18
- net Net-(U10-GL1): track 11.5 -> 0.00 mm
- net Net-(U5-GL1): track 10.6 -> 0.00 mm
- net /MoteurDroit/SH2: track 27.0 -> 17.3 mm, vias 11 -> 13
- net /R_PH: track 34.1 -> 25.7 mm
- net /MoteurGauche/GH2: track 18.2 -> 10.7 mm
- net /nSLEEP: track 110.5 -> 105.1 mm
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- added copper zone on B.Cu, net /MoteurDroit/SH1
- added copper zone on B.Cu, net /MoteurDroit/SH2
- added copper zone on B.Cu, net /MoteurGauche/SH1
- added copper zone on B.Cu, net /MoteurGauche/SH2
- added copper zone on In2.Cu, net GND
- added copper zone on B.Cu, net VDC
- removed copper zone on In2.Cu, net /MoteurDroit/SH1
- removed copper zone on In2.Cu, net /MoteurDroit/SH2
- removed copper zone on F.Cu, net /MoteurDroit/jonctionSS
- removed copper zone on In2.Cu, net /MoteurDroit/jonctionSS
- removed copper zone on In2.Cu, net /MoteurGauche/SH1
- removed copper zone on In2.Cu, net /MoteurGauche/SH2
- removed copper zone on F.Cu, net /MoteurGauche/jonctionSS
- removed copper zone on In2.Cu, net /MoteurGauche/jonctionSS
- removed copper zone on In2.Cu, net VDC
Other:
- board text added: "Driver Moteurs DC avec asservissement Supporte jusqu'à 40V, 15A Encodeur 5V (ENX 10 EASY)"

Commit message: final push
Parts:
- added C32: 18p, Capacitor_SMD:C_0603_1608Metric, F.Cu at (132.7, 80.3)
- added C33: 18p, Capacitor_SMD:C_0603_1608Metric, F.Cu at (132.7, 83.9)
- added U17: ~, Oscillator:WE-XTAL Quartz Crystal 8MHz, F.Cu at (128.8, 81.8)
- moved C9 15.4 mm to (159.6, 93.0), turned to 0 degrees
- moved D2 14.9 mm to (158.1, 89.4), turned to 180 degrees
- moved R12 12.1 mm to (153.0, 90.3), turned to -90 degrees
- moved C28 1.10 mm to (136.0, 81.7)
Connections:
- U16 pad 23: /Px -> unconnected-(U16-PA7-Pad23)
- U16 pad 35: unconnected-(U16-PB14-Pad35) -> /Px
- U16 pad 5: unconnected-(U16-PF0-Pad5) -> /STM_et_Osc/Osc_IN
- U16 pad 6: unconnected-(U16-PF1-Pad6) -> /STM_et_Osc/Osc_OUT
Routing:
- net GND: track 19.4 -> 56.4 mm, vias 403 -> 405
- net /STM_et_Osc/Osc_OUT: track 0.00 -> 12.4 mm
- net /STM_et_Osc/Osc_IN: track 0.00 -> 10.4 mm
- net /Px: track 12.7 -> 3.69 mm, vias 2 -> 0
- net /STM_et_Osc/USART2_RX: track 37.3 -> 44.4 mm
- net /STM_et_Osc/USART2_TX: track 33.6 -> 38.3 mm
- net /STM_et_Osc/NRST: track 34.6 -> 39.1 mm
- net /L_ENCA: track 23.8 -> 25.7 mm
- net /L_ENCB: track 26.5 -> 28.2 mm
- net /L_ENCI: track 28.0 -> 29.7 mm
- net /STM_et_Osc/SWDIO: track 24.9 -> 23.8 mm
Other:
- board text added: "Quartz 8 MHz"

Commit message: finalisation V2 -- manque plus que les vias gnd
Parts:
- removed H3, H4: MountingHole_Pad, MountingHole:MountingHole_2.5mm_Pad
- removed TP1, TP2, TP3: TestPoint, TestPoint:TestPoint_Pad_D1.5mm
- C10: footprint Capacitor_SMD:C_0603_1608Metric_Pad1.08x0.95mm_HandSolder -> Capacitor_SMD:C_0402_1005Metric; moved to F.Cu
- R11: footprint Resistor_SMD:R_0402_1005Metric -> Resistor_SMD:R_0603_1608Metric
- R12: footprint Resistor_SMD:R_0603_1608Metric_Pad0.98x0.95mm_HandSolder -> Resistor_SMD:R_0402_1005Metric
- R13, R14: footprint Resistor_SMD:R_0603_1608Metric_Pad0.98x0.95mm_HandSolder -> Resistor_SMD:R_0402_1005Metric; moved to F.Cu
- U15: footprint BoutonSMD:wurth_pushButton_SMD -> switch:WS-TASU SMT Tact Switch 4.7x3.5 mm side push
- moved J4 105.4 mm to (88.3, 63.6), turned to 90 degrees
- moved U7 98.6 mm to (94.5, 59.5), turned to 0 degrees
- moved H2 98.3 mm to (88.8, 84.8), turned to 180 degrees
- moved U9 89.0 mm to (98.4, 63.1), turned to 180 degrees
- moved J5 86.4 mm to (179.3, 63.6), turned to 90 degrees
- moved U6 79.0 mm to (107.5, 59.5), turned to 90 degrees
- moved G*** 78.7 mm to (125.6, 41.6)
- moved H1 78.2 mm to (178.8, 84.8), turned to 180 degrees
- moved U14 76.9 mm to (172.5, 62.3), turned to 180 degrees
- moved R11 76.7 mm to (85.3, 75.2)
- moved D1 76.7 mm to (85.3, 71.6)
- moved J3 75.3 mm to (108.7, 84.7), turned to 90 degrees
- moved C15 74.6 mm to (111.5, 60.8), turned to 90 degrees
- moved U12 73.2 mm to (168.7, 59.7), turned to 0 degrees
- moved C14 72.8 mm to (113.0, 60.8), turned to -90 degrees
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- renumbered C33 to C32, C32 to C33, C7 to C5, C5 to C7, R4 to R2, R2 to R3, R3 to R4
Connections:
- C7 pad 2: Net-(U2-Vcc) -> GND
- U15 pad 1: GND -> unconnected-(U15-Pad1)
- U15 pad 2: unconnected-(U15-Pad2) -> GND
- U2 pad 14: Net-(U2-Vcc) -> +3.3V
- U3 pad 1: /R_ChA/ -> /R_ChB/
- U3 pad 10: unconnected-(U3-3A-Pad10) -> /R_ChA
- U3 pad 11: unconnected-(U3-3Y-Pad11) -> /R_ENCA
- U3 pad 2: /R_ChA -> /R_ChB
- U3 pad 3: /R_ENCA -> /R_ENCB
- U3 pad 5: /R_ENCB -> unconnected-(U3-2Y-Pad5)
- U3 pad 6: /R_ChB -> unconnected-(U3-2A-Pad6)
- U3 pad 7: /R_ChB/ -> unconnected-(U3-2B-Pad7)
- U3 pad 9: unconnected-(U3-3B-Pad9) -> /R_ChA/
Routing:
- net +5V: track 21.3 -> 80.5 mm, vias 4 -> 10
- net Net-(J9-Pin_4): track 2.50 -> 42.9 mm
- net Net-(J9-Pin_3): track 2.50 -> 41.9 mm
- net Net-(J9-Pin_1): track 2.50 -> 41.3 mm
- net Net-(J9-Pin_2): track 2.50 -> 41.2 mm
- net /STM_et_Osc/Usart3_TX: track 36.1 -> 2.67 mm, vias 2 -> 0
- net /STM_et_Osc/Usart3_RX: track 35.7 -> 2.67 mm, vias 2 -> 0
- net /STM_et_Osc/Uart4_TX: track 30.5 -> 4.06 mm
- net /STM_et_Osc/Uart4_RX: track 29.4 -> 3.48 mm
- net /STM_et_Osc/SWCLK: track 24.7 -> 47.7 mm, vias 0 -> 2
- net /STM_et_Osc/SWDIO: track 23.8 -> 46.0 mm
- net VDC: track 5.98 -> 25.2 mm, vias 39 -> 1
- net /STM_et_Osc/NRST: track 39.1 -> 57.1 mm, vias 3 -> 0
- net /nSLEEP: track 105.1 -> 87.5 mm, vias 3 -> 2
- net /L_ChA/: track 27.1 -> 11.4 mm
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- added copper zone on F.Cu, net +5V
Other:
- board size 92 x 61 mm -> 100 x 40 mm
- board text added: "+"
- board text added: "-"
- board text added: "Boot"
- board text added: "By C. Janus"
- board text added: "Encoder"
- board text added: "GPIO/3.3V/GND"
- board text added: "Left Motor"
- board text added: "Motors ON"
- board text added: "Motors Switch"
- board text added: "Right Motor"
- board text added: "UARTS"
- board text added: "Vbat"
- board text removed: "3V3"
- board text removed: "Battery Level"
- board text removed: "Driver Moteurs DC avec asservissement Supporte jusqu'à 40V, 15A Encodeur 5V (ENX 10 EASY)"
- board text removed: "Encoder_IN"
- board text removed: "GND"
- board text removed: "GPIO"
- board text removed: "MADE IN ARES"
- board text removed: "Made by C.Janus"
- board text removed: "ON/OFF_Motors"
- board text removed: "Quartz 8 MHz"
- board text removed: "UART"

Commit message: finalisation PCB v2
Parts:
- moved G*** 58.6 mm to (170.2, 73.9)
- moved G*** 15.2 mm to (117.1, 54.3)
- moved U15 11.6 mm to (169.6, 87.7)
- moved J2 7.23 mm to (159.0, 84.7)
- moved R10 7.23 mm to (165.7, 79.8)
- moved R8 7.23 mm to (162.0, 79.8)
- moved R9 7.23 mm to (156.9, 79.8)
- moved U4 7.23 mm to (159.7, 74.4)
- moved C5 5.59 mm to (152.5, 74.0)
- moved C27 5.59 mm to (152.5, 76.0)
- moved C32 0.65 mm to (150.1, 78.7)
- moved C33 0.65 mm to (146.8, 78.7)
- moved U17 0.65 mm to (148.5, 82.5)
- moved J11 0.11 mm to (125.6, 82.6)
Connections:
- U15 pad 1: unconnected-(U15-Pad1) -> /STM_et_Osc/NRST
- U15 pad 2: GND -> unconnected-(U15-Pad2)
- U15 pad 3: /STM_et_Osc/NRST -> unconnected-(U15-Pad3)
- U15 pad 4: unconnected-(U15-Pad4) -> GND
Routing:
- net /STM_et_Osc/NRST: track 57.1 -> 67.8 mm
- net /L_ENCI: track 28.6 -> 21.3 mm
- net /L_ENCB: track 26.7 -> 19.4 mm
- net /L_ENCA: track 23.7 -> 16.5 mm
- net /STM_et_Osc/SWDIO: track 46.0 -> 50.4 mm
- net +5V: track 80.5 -> 76.5 mm
- net /STM_et_Osc/SWCLK: track 47.7 -> 51.1 mm
- net /L_ChI: track 14.6 -> 17.3 mm
- net +3.3V: track 34.3 -> 32.3 mm
- net Net-(J9-Pin_2): track 41.2 -> 40.0 mm, vias 0 -> 1
- net /nSLEEP: track 87.5 -> 86.3 mm
- net /STM_et_Osc/USART2_TX: track 35.4 -> 36.6 mm
- net Net-(J9-Pin_1): track 41.3 -> 40.4 mm, vias 0 -> 1
- net /MoteurGauche/GL2: track 16.0 -> 16.8 mm
- net /STM_et_Osc/Osc_OUT: track 14.2 -> 13.5 mm
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Other:
- board text added: "A R E S"
- board text added: "By C.Janus"
- board text removed: "By C. Janus"

Commit message: Final push
Routing:
- net +3.3V: track 32.3 -> 32.8 mm
- net /MoteurDroit/GH2: track 15.6 -> 15.1 mm
- net VDC: track 25.2 -> 25.5 mm, vias 54 -> 69
- net GND: vias 282 -> 310
Other:
- board text added: "Brushed DC Motors driver"

Commit message: Final push
Parts:
- turned R6 to 90 degrees
Routing:
- net GND: track 50.6 -> 59.2 mm, vias 310 -> 309
- net +3.3V: track 32.8 -> 39.3 mm, vias 22 -> 20
- net +5V: track 76.1 -> 73.5 mm, vias 10 -> 8
- net /R_ENCA: track 25.1 -> 27.1 mm
- net /MoteurGauche/GL2: track 16.8 -> 18.7 mm
- net /R_ENCI: track 22.8 -> 24.7 mm
- net /MoteurGauche/GH2: track 10.9 -> 12.7 mm
- net /L_DIR_IN: track 21.0 -> 22.4 mm
- net Net-(J11-Pin_2): track 15.0 -> 16.4 mm
- net Net-(U5-AVDD): track 13.4 -> 14.5 mm
- net /R_DIR_IN: track 17.6 -> 16.7 mm
- net Net-(J11-Pin_1): track 14.2 -> 15.0 mm
- net /STM_et_Osc/USART2_TX: track 36.7 -> 35.8 mm
- net /MoteurDroit/SH2: track 17.4 -> 18.1 mm
- net Net-(U10-CPL): track 8.75 -> 9.41 mm
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
Commit message: Final push
Routing:
- net Net-(U5-AVDD): track 14.5 -> 15.7 mm
- net Net-(U5-DVDD): track 10.4 -> 10.9 mm
Changed lines of the file:
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@@
 	)
 	(via
-		(at 157.59 61.49)
+		(at 156.99 61.52)
 		(size 0.45)
 		(drill 0.3)
@@
 		(net 65)
 	)
+	(segment
+		(start 116.844503 65.724503)
+		(end 116.844503 65.735497)
+		(width 0.25)
+		(layer "F.Cu")
+		(net 65)
+	)
+	(segment
+		(start 116.46 65.34)
+		(end 116.844503 65.724503)
+		(width 0.25)
+		(layer "F.Cu")
+		(net 65)
+	)
+	(segment
+		(start 116.844503 65.735497)
+		(end 116.77 65.81)
+		(width 0.25)
+		(layer "F.Cu")
+		(net 65)
+	)
 	(via
-		(at 116.79 65.81)
+		(at 116.46 65.34)
 		(size 0.45)
 		(drill 0.3)
@@
 	(segment
 		(start 110.39 66.31)
-		(end 116.29 66.31)
+		(end 109.46 65.38)
 		(width 0.25)
 		(layer "In2.Cu")
@@
 	)
 	(segment
-		(start 109.46 63.73)
-		(end 109.46 65.38)
+		(start 115.48 66.31)
+		(end 110.39 66.31)
 		(width 0.25)
 		(layer "In2.Cu")
@@
 	)
 	(segment
-		(start 109.48 63.71)
-		(end 109.46 63.73)
+		(start 116.45 65.34)
+		(end 115.48 66.31)
+		(width 0.25)
+		(layer "In2.Cu")
+		(net 65)
+	)
+	(segment
+		(start 116.46 65.34)
+		(end 116.45 65.34)
 		(width 0.25)
 		(layer "In2.Cu")
@@
 	(segment
 		(start 109.46 65.38)
-		(end 110.39 66.31)
+		(end 109.46 63.73)
 		(width 0.25)
 		(layer "In2.Cu")
@@
 	)
 	(segment
-		(start 116.29 66.31)
-		(end 116.79 65.81)
+		(start 109.46 63.73)
+		(end 109.48 63.71)
 		(width 0.25)
 		(layer "In2.Cu")
@@
 	)
 	(segment
+		(start 117.35 64.62)
+		(end 116.78 64.62)
+		(width 0.25)
+		(layer "F.Cu")
+		(net 66)
+	)
+	(segment
+		(start 116.78 64.62)
+		(end 116.77 64.61)
+		(width 0.25)
+		(layer "F.Cu")
+		(net 66)
+	)
+	(segment
 		(start 110.265 63.21)
 		(end 109.15 63.21)
@@
 	)
 	(via
-		(at 116.81 64.61)
+		(at 117.35 64.62)
 		(size 0.45)
 		(drill 0.3)
@@
 	)
 	(segment
-		(start 110.29 62.16)
-		(end 110.69 62.56)
+		(start 114.29 64.11)
+		(end 114.29 63.51)
 		(width 0.25)
 		(layer "In2.Cu")
@@
 	)
 	(segment
-		(start 110.69 62.56)
+		(start 114.29 63.51)
 		(end 113.34 62.56)
 		(width 0.25)
@@
 	)
 	(segment
-		(start 114.29 63.51)
+		(start 114.79 64.61)
 		(end 114.29 64.11)
 		(width 0.25)
@@
 	)
 	(segment
-		(start 114.79 64.61)
-		(end 116.81 64.61)
+		(start 117.35 64.62)
+		(end 117.34 64.61)
 		(width 0.25)
 		(layer "In2.Cu")
@@
 	)
 	(segment
-		(start 110.27 62.16)
-		(end 110.29 62.16)
+		(start 110.29 62.16)
+		(end 110.27 62.16)
 		(width 0.25)
 		(layer "In2.Cu")
@@
 	)
 	(segment
-		(start 114.29 64.11)
+		(start 117.34 64.61)
 		(end 114.79 64.61)
 		(width 0.25)
@@
 	)
 	(segment
+		(start 110.69 62.56)
+		(end 110.29 62.16)
+		(width 0.25)
+		(layer "In2.Cu")
+		(net 66)
+	)
+	(segment
 		(start 113.34 62.56)
-		(end 114.29 63.51)
+		(end 110.69 62.56)
 		(width 0.25)
 		(layer "In2.Cu")

Commit message: alignement des drv
Parts:
- moved C16 6.51 mm to (109.9, 60.4)
- moved U13 3.30 mm to (162.7, 64.6)
- moved U8 3.18 mm to (104.9, 64.6)
- moved U6 3.13 mm to (104.9, 57.8)
- moved U7 3.00 mm to (97.1, 57.9)
- moved U11 2.97 mm to (162.7, 57.7)
- moved U14 2.92 mm to (170.5, 64.4)
- moved U12 2.56 mm to (170.5, 57.9)
- moved U9 1.82 mm to (97.1, 64.4)
- moved C11 0.84 mm to (116.3, 66.7)
- moved C12 0.84 mm to (116.3, 65.5)
- moved C13 0.84 mm to (116.3, 64.2)
- moved U5 0.84 mm to (112.1, 65.4)
- moved C14 0.19 mm to (112.8, 60.8)
- moved C15 0.11 mm to (111.6, 60.8)
Routing:
- net +5V: track 73.5 -> 67.8 mm
- net /MoteurDroit/SH1: track 14.0 -> 15.3 mm, vias 13 -> 17
- net /MoteurDroit/SH2: track 18.1 -> 19.1 mm, vias 14 -> 17
- net Net-(U5-CPL): track 5.35 -> 6.34 mm
- net Net-(U5-VCP): track 1.22 -> 2.14 mm
- net GND: track 59.2 -> 60.1 mm, vias 309 -> 327
- net /MoteurGauche/GH1: track 15.6 -> 16.4 mm
- net /nSLEEP: track 86.7 -> 85.9 mm
- net /MoteurGauche/GL2: track 18.7 -> 18.0 mm
- net /MoteurGauche/GH2: track 12.7 -> 13.5 mm
- net VDC: track 25.5 -> 26.2 mm, vias 58 -> 57
- net /MoteurDroit/GH2: track 15.3 -> 15.8 mm
- net /MoteurDroit/GL1: track 18.9 -> 19.3 mm, vias 0 -> 2
- net /MoteurGauche/SH1: track 8.49 -> 8.75 mm, vias 12 -> 15
