File: MCU.kicad_sch (KiCad schematic)
At the start: 17 parts, among them J7 Conn_ST_STDC14, U10 STM32F303RETx

Commit message: finalisation schematique
Parts:
- added J1, J12: Conn_01x03, Connector_JST:JST_PH_B3B-PH-K_1x03_P2.00mm_Vertical, symbol Connector_Generic:Conn_01x03
- added J10, J11, J8, J9: Conn_01x04, Connector_PinHeader_2.54mm:PinHeader_1x04_P2.54mm_Vertical, symbol Connector_Generic:Conn_01x04
- added R18, R19, R20, R21: 220, Resistor_SMD:R_0603_1608Metric_Pad0.98x0.95mm_HandSolder, symbol Device:R
Connections:
- net +3.3V: now also J11.1 (Pin_1), J11.2 (Pin_2), J11.3 (Pin_3), J11.4 (Pin_4)
- net ADC3_IN5: now also U10.34 (PB13); no longer U10.57 (PB5)
- net GND: now also J1.3 (Pin_3), J12.3 (Pin_3), J9.1 (Pin_1), J9.2 (Pin_2), J9.3 (Pin_3), J9.4 (Pin_4)
- net L_DIR: now also U10.11 (PC3); no longer U10.42 (PA9)
- net L_PWM: now also U10.37 (PC6); no longer U10.44 (PA11)
- net R_DIR: now also U10.42 (PA9); no longer U10.43 (PA10)
- net R_Enc_A: now also U10.44 (PA11); no longer U10.37 (PC6)
- net R_Enc_B: now also U10.20 (PA4); no longer U10.24 (PC4)
- net R_Enc_I: now also U10.45 (PA12); no longer U10.23 (PA7)
- net R_PWM: now also U10.38 (PC7); no longer U10.45 (PA12)
- net Uart4_TX: now reaches U10.51 (PC10)
- net Uart4_TX: now also R18.1
- net Uart4_RX: now reaches U10.52 (PC11)
- net Uart4_RX: now also R19.1
- net PC12: now reaches U10.53 (PC12)
- net PC12: now also J8.4 (Pin_4)
- net PD2: now reaches U10.54 (PD2)
- net PD2: now also J8.3 (Pin_3)
- net PB3: now reaches U10.55 (PB3)
- net PB3: now also J8.1 (Pin_1)
- net PB4: now reaches U10.56 (PB4)
- net PB4: now also J8.2 (Pin_2)
- net Usart3_RX: now reaches U10.61 (PB8)
- net Usart3_RX: now also R21.1
- net Usart3_TX: now reaches U10.62 (PB9)
- net Usart3_TX: now also R20.1
- new net: J12.1 (Pin_1), R20.2
- new net: J12.2 (Pin_2), R21.2
- new net: J1.2 (Pin_2), R19.2
- new net: J1.1 (Pin_1), R18.2
- new net +5V: J10.1 (Pin_1), J10.2 (Pin_2), J10.3 (Pin_3), J10.4 (Pin_4)
- no-connect marks 35 -> 27
Other:
- note added: "Communication avec UART"
- note added: "Pins GPIO/Usart1/TIM..."
- moved on the sheet: C18, C19, J7, U9

Commit message: reintroduction des mosfet (au lieu des demi-ponts en H), début routage
Parts:
- removed TP4: TestPoint, TestPoint:TestPoint_Pad_D1.5mm, symbol Connector:TestPoint
- added R20, R21, R22, R23: 220, Resistor_SMD:R_0402_1005Metric, symbol Device:R
- C20: footprint Capacitor_SMD:C_0805_2012Metric -> Capacitor_SMD:C_0402_1005Metric
- R18, R19: footprint Resistor_SMD:R_0603_1608Metric_Pad0.98x0.95mm_HandSolder -> Resistor_SMD:R_0402_1005Metric
- R24: renamed from R20; footprint Resistor_SMD:R_0603_1608Metric_Pad0.98x0.95mm_HandSolder -> Resistor_SMD:R_0402_1005Metric
- R25: renamed from R21; footprint Resistor_SMD:R_0603_1608Metric_Pad0.98x0.95mm_HandSolder -> Resistor_SMD:R_0402_1005Metric
- renumbered J8 to J10, J9 to J11, J11 to J6, J10 to J7, J7 to J8, J1 to J9, U9 to U13, U13 to U14, U10 to U15
Connections:
- net PB3: now also R21.1; no longer J10.1 (Pin_1)
- net PB4: now also R20.1; no longer J10.2 (Pin_2)
- net PC12: now also R23.1; no longer J10.4 (Pin_4)
- net PD2: now also R22.1; no longer J10.3 (Pin_3)
- new net: J10.3 (Pin_3), R22.2
- new net: J10.2 (Pin_2), R21.2
- new net: J10.1 (Pin_1), R20.2
- new net: J10.4 (Pin_4), R23.2
Other:
- moved on the sheet: J10, J11, J6, J7

Commit message: maj PCB
Parts:
- removed C18, C19: 18p, Capacitor_SMD:C_0402_1005Metric, symbol Device:C
- removed J7: Conn_01x04, Connector_PinHeader_2.54mm:PinHeader_1x04_P2.54mm_Vertical, symbol Connector_Generic:Conn_01x04
- removed U13: ~, Oscillator:CFPX-104-8MHz_oscillator, symbol CFPX-104-oscillator:CFPX-104-8MHz-wurth
Connections:
- net Usart3_RX: now also R24.1; no longer R25.1
- net Usart3_TX: now also R25.1; no longer R24.1
Other:
- note removed: "Crystal 8MHz"
- moved on the sheet: J10, J11, J12, J6, J8, J9, R18, R19, R20, R21, R22, R23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

Commit message: finalisation PCB
Parts:
- renumbered C20 to C23, C21 to C24, C22 to C25, C23 to C26, C24 to C27, C25 to C28, C26 to C29, C27 to C30, C28 to C31, J11 to J10, J12 to J11, J8 to J7, J9 to J8, J10 to J9, R18 to R15, R19 to R16, R20 to R17, R21 to R18, R22 to R19, R23 to R20, R24 to R21, R25 to R22, U14 to U15, U15 to U16
Connections:
- net R_Enc_B: now also U16.45 (PA12); no longer U16.20 (PA4)
- net R_Enc_I: now also U16.43 (PA10); no longer U16.45 (PA12)
- net SWCLK: now also J7.6 (JCLK/SWCLK); no longer J7.4 (JTMS/SWDIO)
- net SWDIO: now also J7.4 (JTMS/SWDIO); no longer J7.6 (JCLK/SWCLK)
- net PA7: now reaches U16.23 (PA7)
- net ADC3_IN5: no longer names the net of U16.34 (PB13)
- net EXTI14: no longer names the net of U16.3 (PC14)
- net EXTI15: no longer names the net of U16.4 (PC15)
- net EXTI8: no longer names the net of U16.39 (PC8)
- net EXTI9: no longer names the net of U16.40 (PC9)
- net Osc_In: no longer names the net of U16.5 (PF0)
- net Osc_Out: no longer names the net of U16.6 (PF1)
- no-connect marks 27 -> 33

Commit message: final push
Parts:
- added C32, C33: 18p, Capacitor_SMD:C_0603_1608Metric, symbol Device:C
- added U17: ~, Oscillator:WE-XTAL Quartz Crystal 8MHz, symbol CFPX-104-oscillator:CFPX-104-8MHz-wurth
Connections:
- net GND: now also C32.1, C33.2, U17.2 (GND&Lid), U17.4 (GND&Lid)
- net PB14: now reaches U16.35 (PB14)
- net Osc_IN: now reaches U16.5 (PF0)
- net Osc_IN: now also C32.2, U17.3 (Crystal)
- net Osc_OUT: now reaches U16.6 (PF1)
- net Osc_OUT: now also C33.1, U17.1 (Crystal)
- net PA7: no longer names the net of U16.23 (PA7)
- no-connect marks 33 -> 31
Other:
- moved on the sheet: C27, U15

Commit message: finalisation V2 -- manque plus que les vias gnd
Parts:
- U15: footprint BoutonSMD:wurth_pushButton_SMD -> switch:WS-TASU SMT Tact Switch 4.7x3.5 mm side push
- renumbered C33 to C32, C32 to C33
Connections:
- net GND: now also U15.2; no longer U15.1
Changed lines of the file:
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@@
 	)
 	(no_connect
+		(at 133.35 49.53)
+	)
+	(no_connect
 		(at 189.23 118.11)
 	)
@@
 	)
 	(no_connect
-		(at 125.73 49.53)
-	)
-	(no_connect
 		(at 189.23 87.63)
 	)
@@
 	(wire
 		(pts
-			(xy 135.89 52.07) (xy 133.35 52.07)
-		)
-		(stroke
-			(width 0)
-			(type default)
-		)
-	)
-	(wire
-		(pts
 			(xy 50.8 76.2) (xy 52.07 76.2)
 		)
@@
 	(wire
 		(pts
-			(xy 133.35 49.53) (xy 133.35 52.07)
-		)
-		(stroke
-			(width 0)
-			(type default)
-		)
-	)
-	(wire
-		(pts
 			(xy 222.25 90.17) (xy 222.25 82.55)
 		)
@@
 	(wire
 		(pts
+			(xy 125.73 52.07) (xy 125.73 49.53)
+		)
+		(stroke
+			(width 0)
+			(type default)
+		)
+	)
+	(wire
+		(pts
 			(xy 264.16 67.31) (xy 261.62 67.31)
 		)
@@
 	(wire
 		(pts
+			(xy 125.73 52.07) (xy 135.89 52.07)
+		)
+		(stroke
+			(width 0)
+			(type default)
+		)
+	)
+	(wire
+		(pts
 			(xy 31.75 100.33) (xy 41.91 100.33)
 		)
@@
 		(dnp no)
 		(fields_autoplaced yes)
-		(property "Reference" "#PWR057"
+		(property "Reference" "#PWR059"
 			(at 82.55 111.76 0)
 			(effects
@@
 			(project "DRV8701_2Motors"
 				(path "/13741122-7bf4-473f-b117-422f29fb3018/f1aa3c35-e448-45df-a2a6-53fe6f76afb0"
-					(reference "#PWR057")
+					(reference "#PWR059")
 					(unit 1)
 				)
@@
 		(dnp no)
 		(fields_autoplaced yes)
-		(property "Reference" "#PWR066"
+		(property "Reference" "#PWR068"
 			(at 261.62 60.96 0)
 			(effects
@@
 			(project "DRV8701_2Motors"
 				(path "/13741122-7bf4-473f-b117-422f29fb3018/f1aa3c35-e448-45df-a2a6-53fe6f76afb0"
-					(reference "#PWR066")
+					(reference "#PWR068")
 					(unit 1)
 				)
@@
 		(dnp no)
 		(fields_autoplaced yes)
-		(property "Reference" "#PWR053"
+		(property "Reference" "#PWR055"
 			(at 49.53 111.76 0)
 			(effects
@@
 			(project ""
 				(path "/13741122-7bf4-473f-b117-422f29fb3018/f1aa3c35-e448-45df-a2a6-53fe6f76afb0"
-					(reference "#PWR053")
+					(reference "#PWR055")
 					(unit 1)
 				)
@@
 		(dnp no)
 		(fields_autoplaced yes)
-		(property "Reference" "#PWR059"
+		(property "Reference" "#PWR061"
 			(at 113.03 43.18 0)
 			(effects
@@
 			(project "DRV8701_2Motors"
 				(path "/13741122-7bf4-473f-b117-422f29fb3018/f1aa3c35-e448-45df-a2a6-53fe6f76afb0"
-					(reference "#PWR059")
+					(reference "#PWR061")
 					(unit 1)
 				)
@@
 			)
 		)
-		(property "Footprint" "BoutonSMD:wurth_pushButton_SMD"
+		(property "Footprint" "switch:WS-TASU SMT Tact Switch 4.7x3.5 mm side push"
 			(at 129.54 46.99 0)
 			(effects
@@
 		(dnp no)
 		(fields_autoplaced yes)
-		(property "Reference" "#PWR056"
+		(property "Reference" "#PWR058"
 			(at 78.74 166.37 0)
 			(effects
@@
 			(project "DRV8701_2Motors"
 				(path "/13741122-7bf4-473f-b117-422f29fb3018/f1aa3c35-e448-45df-a2a6-53fe6f76afb0"
-					(reference "#PWR056")
+					(reference "#PWR058")
 					(unit 1)
 				)
@@
 		(on_board yes)
 		(dnp no)
-		(property "Reference" "#PWR052"
+		(property "Reference" "#PWR054"
 			(at 43.18 133.35 0)
 			(effects
@@
 			(project ""
 				(path "/13741122-7bf4-473f-b117-422f29fb3018/f1aa3c35-e448-45df-a2a6-53fe6f76afb0"
-					(reference "#PWR052")
+					(reference "#PWR054")
 					(unit 1)
 				)
@@
 		(dnp no)
 		(fields_autoplaced yes)
-		(property "Reference" "#PWR054"
+		(property "Reference" "#PWR056"
 			(at 52.07 82.55 0)
 			(effects
@@
 			(project "DRV8701_2Motors"
 				(path "/13741122-7bf4-473f-b117-422f29fb3018/f1aa3c35-e448-45df-a2a6-53fe6f76afb0"
-					(reference "#PWR054")
+					(reference "#PWR056")
 					(unit 1)
 				)
@@
 		(on_board yes)
 		(dnp no)
-		(property "Reference" "#PWR062"
+		(property "Reference" "#PWR064"
 			(at 179.07 33.02 0)
 			(effects
@@
 			(project "DRV8701_2Motors"
 				(path "/13741122-7bf4-473f-b117-422f29fb3018/f1aa3c35-e448-45df-a2a6-53fe6f76afb0"
-					(reference "#PWR062")
+					(reference "#PWR064")
 					(unit 1)
 				)
@@
 		(dnp no)
 		(fields_autoplaced yes)
-		(property "Reference" "#PWR064"
+		(property "Reference" "#PWR066"
 			(at 204.47 33.02 0)
 			(effects
@@
 			(project "DRV8701_2Motors"
 				(path "/13741122-7bf4-473f-b117-422f29fb3018/f1aa3c35-e448-45df-a2a6-53fe6f76afb0"
-					(reference "#PWR064")
+					(reference "#PWR066")
 					(unit 1)
 				)
@@
 		(dnp no)
 		(fields_autoplaced yes)
-		(property "Reference" "C33"
+		(property "Reference" "C32"
 			(at 226.06 92.7099 0)
 			(effects
@@
 			(project "DRV8701_2Motors"
 				(path "/13741122-7bf4-473f-b117-422f29fb3018/f1aa3c35-e448-45df-a2a6-53fe6f76afb0"
-					(reference "C33")
+					(reference "C32")
 					(unit 1)
 				)
@@
 		(dnp no)
 		(fields_autoplaced yes)
-		(property "Reference" "#PWR063"
+		(property "Reference" "#PWR065"
 			(at 189.23 43.18 0)
 			(effects
@@
 			(project "DRV8701_2Motors"
 				(path "/13741122-7bf4-473f-b117-422f29fb3018/f1aa3c35-e448-45df-a2a6-53fe6f76afb0"
-					(reference "#PWR063")
+					(reference "#PWR065")
 					(unit 1)
 				)
@@
 		(dnp no)
 		(fields_autoplaced yes)
-		(property "Reference" "#PWR065"
+		(property "Reference" "#PWR067"
 			(at 237.49 106.68 0)
 			(effects
@@
 			(project "DRV8701_2Motors"
 				(path "/13741122-7bf4-473f-b117-422f29fb3018/f1aa3c35-e448-45df-a2a6-53fe6f76afb0"
-					(reference "#PWR065")
+					(reference "#PWR067")
 					(unit 1)
 				)
@@
 		(dnp no)
 		(fields_autoplaced yes)
-		(property "Reference" "#PWR061"
+		(property "Reference" "#PWR063"
 			(at 172.72 140.97 0)
 			(effects
@@
 			(project "DRV8701_2Motors"
 				(path "/13741122-7bf4-473f-b117-422f29fb3018/f1aa3c35-e448-45df-a2a6-53fe6f76afb0"
-					(reference "#PWR061")
+					(reference "#PWR063")
 					(unit 1)
 				)
@@
 		(on_board yes)
 		(dnp no)
-		(property "Reference" "#PWR055"
+		(property "Reference" "#PWR057"
 			(at 53.34 44.45 0)
 			(effects
@@
 			(project "DRV8701_2Motors"
 				(path "/13741122-7bf4-473f-b117-422f29fb3018/f1aa3c35-e448-45df-a2a6-53fe6f76afb0"
-					(reference "#PWR055")
+					(reference "#PWR057")
 					(unit 1)
 				)
@@
 		(dnp no)
 		(fields_autoplaced yes)
-		(property "Reference" "#PWR058"
+		(property "Reference" "#PWR060"
 			(at 113.03 33.02 0)
 			(effects
@@
 			(project "DRV8701_2Motors"
 				(path "/13741122-7bf4-473f-b117-422f29fb3018/f1aa3c35-e448-45df-a2a6-53fe6f76afb0"
-					(reference "#PWR058")
+					(reference "#PWR060")
 					(unit 1)
 				)
@@
 		(dnp no)
 		(fields_autoplaced yes)
-		(property "Reference" "C32"
+		(property "Reference" "C33"
 			(at 267.97 71.1199 0)
 			(effects
@@
 			(project ""
 				(path "/13741122-7bf4-473f-b117-422f29fb3018/f1aa3c35-e448-45df-a2a6-53fe6f76afb0"
-					(reference "C32")
+					(reference "C33")
 					(unit 1)
 				)
@@
 		(dnp no)
 		(fields_autoplaced yes)
-		(property "Reference" "#PWR060"
+		(property "Reference" "#PWR062"
 			(at 135.89 59.69 0)
 			(effects
@@
 			(project "DRV8701_2Motors"
 				(path "/13741122-7bf4-473f-b117-422f29fb3018/f1aa3c35-e448-45df-a2a6-53fe6f76afb0"
-					(reference "#PWR060")
+					(reference "#PWR062")
 					(unit 1)
 				)

Commit message: finalisation PCB v2
Connections:
- net GND: now also U15.4; no longer U15.2
- net NRST: now also U15.1; no longer U15.3
Other:
- moved on the sheet: U15
Changed lines of the file:
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@@
+	)
+	(junction
+		(at 135.89 52.07)
+		(diameter 0)
+		(color 0 0 0 0)
 	)
 	(junction
@@
 	)
 	(junction
-		(at 135.89 52.07)
+		(at 139.7 44.45)
 		(diameter 0)
 		(color 0 0 0 0)
@@
 	)
 	(junction
-		(at 139.7 44.45)
-		(diameter 0)
-		(color 0 0 0 0)
-	)
-	(junction
 		(at 189.23 36.83)
 		(diameter 0)
@@
 	)
 	(no_connect
-		(at 133.35 49.53)
-	)
-	(no_connect
 		(at 189.23 118.11)
 	)
@@
 	)
 	(no_connect
+		(at 125.73 49.53)
+	)
+	(no_connect
 		(at 189.23 87.63)
 	)
 	(no_connect
+		(at 133.35 44.45)
+	)
+	(no_connect
 		(at 66.04 63.5)
 	)
@@
 	)
 	(no_connect
-		(at 125.73 44.45)
-	)
-	(no_connect
 		(at 189.23 57.15)
 	)
@@
 	(wire
 		(pts
+			(xy 125.73 41.91) (xy 139.7 41.91)
+		)
+		(stroke
+			(width 0)
+			(type default)
+		)
+	)
+	(wire
+		(pts
 			(xy 172.72 134.62) (xy 173.99 134.62)
 		)
@@
 	(wire
 		(pts
+			(xy 139.7 41.91) (xy 139.7 44.45)
+		)
+		(stroke
+			(width 0)
+			(type default)
+		)
+	)
+	(wire
+		(pts
+			(xy 133.35 49.53) (xy 133.35 52.07)
+		)
+		(stroke
+			(width 0)
+			(type default)
+		)
+	)
+	(wire
+		(pts
 			(xy 39.37 134.62) (xy 39.37 137.16)
 		)
@@
 	(wire
 		(pts
+			(xy 125.73 44.45) (xy 125.73 41.91)
+		)
+		(stroke
+			(width 0)
+			(type default)
+		)
+	)
+	(wire
+		(pts
 			(xy 222.25 100.33) (xy 237.49 100.33)
 		)
@@
 	(wire
 		(pts
-			(xy 125.73 52.07) (xy 125.73 49.53)
-		)
-		(stroke
-			(width 0)
-			(type default)
-		)
-	)
-	(wire
-		(pts
 			(xy 264.16 67.31) (xy 261.62 67.31)
 		)
@@
 	(wire
 		(pts
-			(xy 133.35 44.45) (xy 139.7 44.45)
-		)
-		(stroke
-			(width 0)
-			(type default)
-		)
-	)
-	(wire
-		(pts
 			(xy 171.45 29.21) (xy 173.99 29.21)
 		)
@@
 	(wire
 		(pts
+			(xy 133.35 52.07) (xy 135.89 52.07)
+		)
+		(stroke
+			(width 0)
+			(type default)
+		)
+	)
+	(wire
+		(pts
 			(xy 77.47 134.62) (xy 80.01 134.62)
 		)
@@
 		(pts
 			(xy 144.78 54.61) (xy 153.67 54.61)
-		)
-		(stroke
-			(width 0)
-			(type default)
-		)
-	)
-	(wire
-		(pts
-			(xy 125.73 52.07) (xy 135.89 52.07)
 		)
 		(stroke
@@
 	(symbol
 		(lib_id "Generic_Switch:Switch_SMD")
-		(at 129.54 46.99 0)
+		(at 129.54 46.99 180)
 		(unit 1)
 		(exclude_from_sim no)
@@
 		(fields_autoplaced yes)
 		(property "Reference" "U15"
-			(at 129.667 40.64 0)
+			(at 129.413 40.64 0)
 			(effects
 				(font
@@
 		)
 		(property "Value" "~"
-			(at 129.667 43.18 0)
-			(effects
-				(font
+			(at 129.413 43.18 0)
+			(effects
+				(font
